File: hw/Score-Board-Digits.kicad_sch (KiCad schematic)
At the start: 33 parts, among them J1 Conn_02x09_Odd_Even

Commit message: PCB routing done
Parts:
- R1, R2, R3, R4, R5, R6, R7: value 0 -> 77
- R10, R11, R12, R13, R14, R15, R16, R9: value 150 -> 100
- R8: value 0 -> 100
Changed lines of the file:
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@@
       (effects (font (size 1.27 1.27)))
     )
-    (property "Value" "0" (at 48.26 72.39 90)
+    (property "Value" "77" (at 48.26 72.39 90)
       (effects (font (size 1.27 1.27)))
     )
@@
       (effects (font (size 1.27 1.27)))
     )
-    (property "Value" "0" (at 48.26 92.71 90)
+    (property "Value" "77" (at 48.26 92.71 90)
       (effects (font (size 1.27 1.27)))
     )
@@
       (effects (font (size 1.27 1.27)))
     )
-    (property "Value" "0" (at 48.26 87.63 90)
+    (property "Value" "77" (at 48.26 87.63 90)
       (effects (font (size 1.27 1.27)))
     )
@@
       (effects (font (size 1.27 1.27)))
     )
-    (property "Value" "150" (at 119.38 165.1 90)
+    (property "Value" "100" (at 119.38 165.1 90)
       (effects (font (size 1.27 1.27)))
     )
@@
       (effects (font (size 1.27 1.27)))
     )
-    (property "Value" "150" (at 119.38 180.34 90)
+    (property "Value" "100" (at 119.38 180.34 90)
       (effects (font (size 1.27 1.27)))
     )
@@
       (effects (font (size 1.27 1.27)))
     )
-    (property "Value" "150" (at 119.38 135.89 90)
+    (property "Value" "100" (at 119.38 135.89 90)
       (effects (font (size 1.27 1.27)))
     )
@@
       (effects (font (size 1.27 1.27)))
     )
-    (property "Value" "150" (at 119.38 140.97 90)
+    (property "Value" "100" (at 119.38 140.97 90)
       (effects (font (size 1.27 1.27)))
     )
@@
       (effects (font (size 1.27 1.27)))
     )
-    (property "Value" "150" (at 119.38 175.26 90)
+    (property "Value" "100" (at 119.38 175.26 90)
       (effects (font (size 1.27 1.27)))
     )
@@
       (effects (font (size 1.27 1.27)))
     )
-    (property "Value" "150" (at 119.38 130.81 90)
+    (property "Value" "100" (at 119.38 130.81 90)
       (effects (font (size 1.27 1.27)))
     )
@@
       (effects (font (size 1.27 1.27)))
     )
-    (property "Value" "0" (at 48.26 102.87 90)
+    (property "Value" "77" (at 48.26 102.87 90)
       (effects (font (size 1.27 1.27)))
     )
@@
       (effects (font (size 1.27 1.27)))
     )
-    (property "Value" "150" (at 119.38 170.18 90)
+    (property "Value" "100" (at 119.38 170.18 90)
       (effects (font (size 1.27 1.27)))
     )
@@
       (effects (font (size 1.27 1.27)))
     )
-    (property "Value" "0" (at 48.26 107.95 90)
+    (property "Value" "100" (at 48.26 107.95 90)
       (effects (font (size 1.27 1.27)))
     )
@@
       (effects (font (size 1.27 1.27)))
     )
-    (property "Value" "0" (at 48.26 97.79 90)
+    (property "Value" "77" (at 48.26 97.79 90)
       (effects (font (size 1.27 1.27)))
     )
@@
       (effects (font (size 1.27 1.27)))
     )
-    (property "Value" "150" (at 119.38 125.73 90)
+    (property "Value" "100" (at 119.38 125.73 90)
       (effects (font (size 1.27 1.27)))
     )
@@
       (effects (font (size 1.27 1.27)))
     )
-    (property "Value" "0" (at 48.26 82.55 90)
+    (property "Value" "77" (at 48.26 82.55 90)
       (effects (font (size 1.27 1.27)))
     )
@@
       (effects (font (size 1.27 1.27)))
     )
-    (property "Value" "0" (at 48.26 77.47 90)
-      (effects (font (size 1.27 1.27)))
-    )
+    (property "Value" "77" (at 48.26 77.47 90)
+      (effects (font (size 1.27 1.27)))
+    )

Commit message: Add pull-down res to segment drives.
Parts:
- R1, R2, R3, R4, R5, R6, R7: value 77 -> 75
Other:
- note added: "Note-1"
Changed lines of the file:
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@@
+    (fill (type none))
+  )
+  (rectangle (start 40.64 69.85) (end 50.8 116.84)
+    (stroke (width 0) (type dash))
     (fill (type none))
   )
@@
     (fill (type none))
   )
+  (text_box "Note-1: R1-R7 Resistance:\n 0: (jumper) For large (5 LEDs/Segment) displays\n75: For medium (3 LEDs/Segment) displays\n R8 is 100, as it is for the decimal point (a single LED)"
+    (at 15.24 189.23 0) (size 59.69 11.43)
+    (stroke (width 0) (type default))
+    (fill (type none))
+    (effects (font (size 1.27 1.27)) (justify left top))
+  )
   (text "(LARGE DIGIT ASSY)" (at 153.67 77.47 0)
     (effects (font (size 1.27 1.27) (color 0 0 255 1)) (justify left bottom))
+  )
+  (text "Note-1" (at 41.91 115.57 0)
+    (effects (font (size 1.27 1.27)) (justify left bottom))
   )
   (text "B" (at 116.84 158.75 0)
@@
       (effects (font (size 1.27 1.27)))
     )
-    (property "Value" "77" (at 48.26 72.39 90)
+    (property "Value" "75" (at 48.26 72.39 90)
       (effects (font (size 1.27 1.27)))
     )
@@
       (effects (font (size 1.27 1.27)))
     )
-    (property "Value" "77" (at 48.26 92.71 90)
+    (property "Value" "75" (at 48.26 92.71 90)
       (effects (font (size 1.27 1.27)))
     )
@@
       (effects (font (size 1.27 1.27)))
     )
-    (property "Value" "77" (at 48.26 87.63 90)
+    (property "Value" "75" (at 48.26 87.63 90)
       (effects (font (size 1.27 1.27)))
     )
@@
       (effects (font (size 1.27 1.27)))
     )
-    (property "Value" "77" (at 48.26 102.87 90)
+    (property "Value" "75" (at 48.26 102.87 90)
       (effects (font (size 1.27 1.27)))
     )
@@
       (effects (font (size 1.27 1.27)))
     )
-    (property "Value" "77" (at 48.26 97.79 90)
+    (property "Value" "75" (at 48.26 97.79 90)
       (effects (font (size 1.27 1.27)))
     )
@@
       (effects (font (size 1.27 1.27)))
     )
-    (property "Value" "77" (at 48.26 82.55 90)
+    (property "Value" "75" (at 48.26 82.55 90)
       (effects (font (size 1.27 1.27)))
     )
@@
       (effects (font (size 1.27 1.27)))
     )
-    (property "Value" "77" (at 48.26 77.47 90)
-      (effects (font (size 1.27 1.27)))
-    )
+    (property "Value" "75" (at 48.26 77.47 90)
+      (effects (font (size 1.27 1.27)))
+    )
